File: Attiny85/Demo/Experimental(Latest_changes)/Therm2Bin_varPWM/at85_Latest/at85_Latest.sch (KiCad schematic (older format))
At the start: 42 parts, among them U1 attiny85_exp, U10 plot_v1, U11 adc_bridge_3, U12 adc_bridge_3, U13 plot_v1, U14 dac_bridge_2, U15 plot_v1, U16 plot_v1, U2 plot_v1, U3 plot_v1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

Commit message: Added limited timer0 functionality
Parts:
- removed U1: attiny85_exp, symbol attiny85_exp
- removed U10, U13, U15, U6: plot_v1, symbol plot_v1
- removed U12: adc_bridge_3, symbol adc_bridge_3
- removed U14: dac_bridge_2, symbol dac_bridge_2
- removed U5: dac_bridge_4, symbol dac_bridge_4
- removed U7: therm2bin2bit, symbol therm2bin2bit
- added U1, U12, U14, U7: plot_v1, symbol plot_v1
- added U10: adc_bridge_3, symbol adc_bridge_3
- added U13: dac_bridge_2, symbol dac_bridge_2
- added U15: dac_bridge_4, symbol dac_bridge_4
- added U5: therm2bin2bit, symbol therm2bin2bit
- added U6: at85_latest, symbol at85_latest
