File: Attiny85/Demo/ATtiny85/attiny85-test/attiny85-test.sch (KiCad schematic (older format))
At the start: 8 parts, among them U1 adc_bridge_2, U3 adc_bridge_1, U4 attiny_85_nghdl, U5 dac_bridge_1, U6 plot_v1

Commit message: New version with timer0 (#52)
Parts:
- v1: symbol DC -> DC-RESCUE-attiny85-test
Changed lines of the file:
@@
 $EndComp
 $Comp
-L DC v1
+L DC-RESCUE-attiny85-test v1
 U 1 1 5E55FCA0
 P 2450 3700
